File: Cosmonode/Cosmonode.sch (KiCad schematic (older format))
At the start: 49 parts, among them J1 CONN_01X12, J10 WEEE_Logo, J11 Aloes_Logo, J12 Aloes_mini_Logo, J13 CONN_01X05, J14 GS2, J2 CONN_01X12, J3 GS2, J4 OSHW, J5 CONN_01X02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

Commit message: start v0.8
Parts:
- R8: value 1M -> 470K
Other:
- note added: "A0 =\nA1 =\nA2 = ATSHA204\nA3 = Battery Report\nA4 = SDA\nA5 = SCL\nA6 = RN2483 Rx LED \nA7 = RN2483 Tx LED\nD0 = RX\nD1 = TX\nD2 = ResetInterrupt ( from RN2483 ) or RFM69 DI0\nD3 = ButtonInterrupt ( ask for config )\nD4 =\nD5 =\nD6 = optionnal GND ( battery level )\nD7 = \nD8 = RN2483 Tx \nD9 = RN2483 Rx - RFM69 Reset\nD10 = RN2483 Reset - RFM69 NSS\nD11 = - RFM69 MOSI\nD12 = RFM69 MISO\nD13 = R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"
- note added: "Cosmonode v0.8\nATmega328p\nRFM69CW or RN 2483 ( both 868Mhz Radio )"
- note removed: "A0 =\nA1 =\nA2 = ATSHA204\nA3 = Battery Report\nA4 = SDA\nA5 = SCL\nA6 = RN2483 Rx LED \nA7 = RN2483 Tx LED\nD0 = RX\nD1 = TX\nD2 = ResetInterrupt ( from RN2483 ) or RFM69 DI0\nD3 = ButtonInterrupt ( ask for config )\nD4 =\nD5 =\nD6 =\nD7 = \nD8 = RN2483 Tx \nD9 = RN2483 Rx - RFM69 Reset\nD10 = RN2483 Reset - RFM69 NSS\nD11 = - RFM69 MOSI\nD12 = RFM69 MISO\nD13 = RFM69 SCK"
- note removed: "Cosmonode v0.7\nATmega328p\nRFM69CW or RN 2483 ( both 868Mhz Radio )"
