File: Cosmonode_ext01/Cosmonode_ext01.sch (KiCad schematic (older format))
At the start: 4 parts, among them J1 CONN_01X04, J2 CONN_01X01, J3 GS3, U1 SI7020-A20-YM0R

Commit message: start v0.8
Parts:
- added C1: 100nF, Capacitors_SMD:C_0603_HandSoldering, symbol C_Small
- added J4, J5, J6: CONN_01X01, Wire_Pads:SolderWirePad_single_1-2mmDrill, symbol CONN_01X01
- J2: footprint Mounting_Holes:MountingHole_2.5mm -> Wire_Pads:SolderWirePad_single_1-2mmDrill
Connections:
- net +3V3: now also C1.1
- net GND: now also C1.2; no longer U1.7 (TGND)
Changed lines of the file:
@@
 LIBS:BMP180
 LIBS:SI7020-A20-YM0R
-LIBS:BME280-cache
+LIBS:Cosmonode_ext01-cache
 EELAYER 25 0
 EELAYER END
@@
 Text GLabel 6150 4200 0    51   BiDi ~ 0
 A5
-$Comp
-L GND #PWR01
-U 1 1 5A2EA769
-P 5850 4100
-F 0 "#PWR01" H 5850 4150 30  0001 C CNN
-F 1 "GND" H 5850 3975 30  0001 C CNN
-F 2 "" H 5850 4100 60  0000 C CNN
-F 3 "" H 5850 4100 60  0000 C CNN
-	1    5850 4100
-	1    0    0    -1
-$EndComp
-$Comp
-L +3V3 #PWR02
-U 1 1 5A2EA79C
-P 6050 4000
-F 0 "#PWR02" H 6050 4225 30  0001 C CNN
-F 1 "+3V3" V 5975 4000 30  0001 C CNN
-F 2 "" H 6050 4000 60  0000 C CNN
-F 3 "" H 6050 4000 60  0000 C CNN
-	1    6050 4000
-	1    0    0    -1
-$EndComp
 Wire Wire Line
 	6050 4000 6150 4000
@@
 A4
 $Comp
-L +3V3 #PWR03
+L +3V3 #PWR01
 U 1 1 5A2EA7E0
 P 5250 3000
-F 0 "#PWR03" H 5250 3225 30  0001 C CNN
+F 0 "#PWR01" H 5250 3225 30  0001 C CNN
 F 1 "+3V3" V 5175 3000 30  0001 C CNN
 F 2 "" H 5250 3000 60  0000 C CNN
@@
 $EndComp
 $Comp
-L GND #PWR04
+L GND #PWR02
 U 1 1 5A2EA7F1
 P 5400 3400
-F 0 "#PWR04" H 5400 3450 30  0001 C CNN
+F 0 "#PWR02" H 5400 3450 30  0001 C CNN
 F 1 "GND" H 5400 3275 30  0001 C CNN
 F 2 "" H 5400 3400 60  0000 C CNN
@@
 $EndComp
 Wire Wire Line
-	5250 3300 5400 3300
-Wire Wire Line
-	5400 3300 5400 3400
+	5400 3250 5400 3400
 Wire Wire Line
 	5400 3400 5250 3400
-$Comp
-L CONN_01X01 J2
-U 1 1 5A2EA9AD
-P 7050 3450
-F 0 "J2" H 7050 3550 50  0000 C CNN
-F 1 "CONN_01X01" V 7150 3450 50  0000 C CNN
-F 2 "Mounting_Holes:MountingHole_2.5mm" H 7050 3450 50  0001 C CNN
-F 3 "" H 7050 3450 50  0001 C CNN
-	1    7050 3450
-	1    0    0    -1
-$EndComp
-NoConn ~ 6850 3450
 $Comp
 L GS3 J3
@@
 $EndComp
 $Comp
-L GND #PWR05
+L GND #PWR03
 U 1 1 5A2EAC3F
 P 3950 4000
-F 0 "#PWR05" H 3950 4050 30  0001 C CNN
+F 0 "#PWR03" H 3950 4050 30  0001 C CNN
 F 1 "GND" H 3950 3875 30  0001 C CNN
 F 2 "" H 3950 4000 60  0000 C CNN
@@
 Wire Wire Line
 	4050 3400 4050 3700
+$Comp
+L C_Small C1
+U 1 1 5A4535B3
+P 5400 3150
+F 0 "C1" H 5410 3220 50  0000 L CNN
+F 1 "100nF" H 5410 3070 50  0000 L CNN
+F 2 "Capacitors_SMD:C_0603_HandSoldering" H 5400 3150 50  0001 C CNN
+F 3 "" H 5400 3150 50  0001 C CNN
+	1    5400 3150
+	1    0    0    -1
+$EndComp
+$Comp
+L SUP_+3V3 #PWR04
+U 1 1 5A453718
+P 6050 4000
+F 0 "#PWR04" H 6050 4225 30  0001 C CNN
+F 1 "SUP_+3V3" V 5975 4000 30  0001 C CNN
+F 2 "" H 5950 4125 60  0001 C CNN
+F 3 "" H 6050 4225 60  0001 C CNN
+	1    6050 4000
+	1    0    0    -1
+$EndComp
+$Comp
+L SUP_GND #PWR05
+U 1 1 5A45375C
+P 5850 4100
+F 0 "#PWR05" H 5850 4150 30  0001 C CNN
+F 1 "SUP_GND" H 5850 3975 30  0001 C CNN
+F 2 "" H 5850 4100 60  0000 C CNN
+F 3 "" H 5850 4100 60  0000 C CNN
+	1    5850 4100
+	1    0    0    -1
+$EndComp
+NoConn ~ 5250 3300
+Wire Wire Line
+	5250 3000 5400 3000
+Wire Wire Line
+	5400 3000 5400 3050
+$Comp
+L CONN_01X01 J2
+U 1 1 5A453B9F
+P 7000 2500
+F 0 "J2" H 7000 2600 50  0000 C CNN
+F 1 "CONN_01X01" V 7100 2500 50  0000 C CNN
+F 2 "Wire_Pads:SolderWirePad_single_1-2mmDrill" H 7000 2500 50  0001 C CNN
+F 3 "" H 7000 2500 50  0001 C CNN
+	1    7000 2500
+	1    0    0    -1
+$EndComp
+$Comp
+L CONN_01X01 J4
+U 1 1 5A453C13
+P 7050 2900
+F 0 "J4" H 7050 3000 50  0000 C CNN
+F 1 "CONN_01X01" V 7150 2900 50  0000 C CNN
+F 2 "Wire_Pads:SolderWirePad_single_1-2mmDrill" H 7050 2900 50  0001 C CNN
+F 3 "" H 7050 2900 50  0001 C CNN
+	1    7050 2900
+	1    0    0    -1
+$EndComp
+$Comp
+L CONN_01X01 J5
+U 1 1 5A453C53
+P 7500 2350
+F 0 "J5" H 7500 2450 50  0000 C CNN
+F 1 "CONN_01X01" V 7600 2350 50  0000 C CNN
+F 2 "Wire_Pads:SolderWirePad_single_1-2mmDrill" H 7500 2350 50  0001 C CNN
+F 3 "" H 7500 2350 50  0001 C CNN
+	1    7500 2350
+	1    0    0    -1
+$EndComp
+$Comp
+L CONN_01X01 J6
+U 1 1 5A453C98
+P 7500 2800
+F 0 "J6" H 7500 2900 50  0000 C CNN
+F 1 "CONN_01X01" V 7600 2800 50  0000 C CNN
+F 2 "Wire_Pads:SolderWirePad_single_1-2mmDrill" H 7500 2800 50  0001 C CNN
+F 3 "" H 7500 2800 50  0001 C CNN
+	1    7500 2800
+	1    0    0    -1
+$EndComp
 $EndSCHEMATC
