File: Cosmonode_ext02/Cosmonode_ext02.kicad_pcb (KiCad board)
At the start: 2 copper layers, 48.3 x 31.8 mm, 23 parts, among them J1 CONN_01X04, J10 CONN_01X06, J2 CONN_01X04, J3 CONN_01X12, J4 CONN_01X12, J5 GS3, J6 GS3, J7 Aloes_Logo, J8 OSHW_Logo, J9 CONN_01X04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

Commit message: start v0.8
Parts:
- added J12: GS3, Connectors:GS3, F.Cu at (184.2, 114.3)
- J10: footprint Pin_Headers:Pin_Header_Straight_1x06_Pitch2.54mm -> Pin_Headers:Pin_Header_Angled_1x06_Pitch2.54mm
- moved J7 1.42 mm to (177.2, 114.3)
- moved J8 1.27 mm to (174.0, 97.8)
Connections:
- J10 pad 3: A4 -> MOSI
- J10 pad 4: A5 -> MISO
- J10 pad 5: D4 -> SCK
- J10 pad 6: D5 -> D4
- J9 pad 1: +3V3 -> Net-(J12-Pad2)
- J9 pad 2: GND -> Net-(C1-Pad1)
Routing:
- net Net-(C1-Pad1): track 0.00 -> 105.1 mm, vias 0 -> 1
- net +3V3: track 0.00 -> 74.5 mm, vias 0 -> 2
- net A4: track 0.00 -> 58.0 mm, vias 0 -> 1
- net A5: track 0.00 -> 53.4 mm, vias 0 -> 1
- net GND: track 0.00 -> 50.3 mm, vias 0 -> 1
- net +5V: track 0.00 -> 44.5 mm, vias 0 -> 2
- net Net-(C1-Pad2): track 0.00 -> 37.6 mm
- net MOSI: track 0.00 -> 37.5 mm
- net MISO: track 0.00 -> 36.5 mm, vias 0 -> 1
- net SCK: track 0.00 -> 35.3 mm
- net A0_5V: track 0.00 -> 28.4 mm
- net Net-(C5-Pad2): track 0.00 -> 22.8 mm
- net D4: track 0.00 -> 20.1 mm
- net D5: track 0.00 -> 19.9 mm, vias 0 -> 1
- net D6: track 0.00 -> 19.8 mm
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- added copper zone on B.Cu, net Net-(C1-Pad1)
- added copper zone on F.Cu, net Net-(C1-Pad1)
Other:
- board text added: "Extension #2 v0.7 Liquid Level XKC-Y25 sensor"
- board text removed: "Extension #2 Liquid Level XKC-Y25 sensor"
